Commit message: reconfiguring remapper for linkages

File: src/jax_description/urdf/const.xacro (robot description, xacro)
@@ -39,9 +39,9 @@
   <xacro:property name="hip_velocity_max" value="30.1"/>
   <xacro:property name="hip_torque_max" value="23.7"/>
-  <xacro:property name="thigh_position_max" value="1.396263"/>
+  <xacro:property name="thigh_position_max" value="1.2"/>
   <xacro:property name="thigh_position_min" value="-1.396263"/>
   <xacro:property name="thigh_velocity_max" value="30.1"/>
   <xacro:property name="thigh_torque_max" value="23.7"/>
-  <xacro:property name="calf_position_max" value="1.047198"/>
+  <xacro:property name="calf_position_max" value="0.95"/>
   <xacro:property name="calf_position_min" value="-1.047198"/>
   <xacro:property name="calf_velocity_max" value="30.1"/>

Commit message: 2

File: src/jax_description/urdf/const.xacro (robot description, xacro)
@@ -43,6 +43,6 @@
   <xacro:property name="thigh_velocity_max" value="30.1"/>
   <xacro:property name="thigh_torque_max" value="23.7"/>
-  <xacro:property name="calf_position_max" value="0.95"/>
-  <xacro:property name="calf_position_min" value="-1.047198"/>
+  <xacro:property name="calf_position_max" value="0.85"/>
+  <xacro:property name="calf_position_min" value="-1.3"/>
   <xacro:property name="calf_velocity_max" value="30.1"/>
   <xacro:property name="calf_torque_max" value="35.55"/>

Commit message: worked on display node

File: src/jax_description/urdf/const.xacro (robot description, xacro)
@@ -39,6 +39,6 @@
   <xacro:property name="hip_velocity_max" value="30.1"/>
   <xacro:property name="hip_torque_max" value="23.7"/>
-  <xacro:property name="thigh_position_max" value="1.2"/>
-  <xacro:property name="thigh_position_min" value="-1.396263"/>
+  <xacro:property name="thigh_position_max" value="1.3"/>
+  <xacro:property name="thigh_position_min" value="-1.3"/>
   <xacro:property name="thigh_velocity_max" value="30.1"/>
   <xacro:property name="thigh_torque_max" value="23.7"/>
